File: Public/Module/RelayModuleMK1/RelayModuleMK1_KiCad/RelayModuleMK1_KiCad.kicad_pcb (KiCad board)
At the start: 2 copper layers, 101.6 x 88.9 mm, 50 parts, among them J1 2EDG-5.08mm_2P, Q1 S9014 SOT23-3, Q2 S9014 SOT23-3, Q3 S9014 SOT23-3, Q4 S9014 SOT23-3, U1 ILQ32, U2 LM339

Commit message: Update RelayModuleMK1
Parts:
- moved D1 0.32 mm to (206.1, 104.8)
- moved JOUT0 0.28 mm to (215.9, 55.9)
- moved JOUT1 0.28 mm to (231.1, 55.9)
- moved JOUT2 0.28 mm to (246.4, 55.9)
- moved JOUT3 0.28 mm to (261.6, 55.9)
Routing:
- net Net-(DA3-A): track 10.0 -> 7.67 mm, vias 1 -> 0
- net Net-(DA2-A): track 10.0 -> 7.67 mm, vias 1 -> 0
- net Net-(DA1-A): track 10.0 -> 7.67 mm, vias 1 -> 0
- net Net-(DA0-A): track 10.0 -> 7.67 mm, vias 1 -> 0
- net VCC_PWR: track 316.0 -> 315.5 mm, vias 2 -> 1
- net GNDPWR: vias 1 -> 5
- added copper zone on B.Cu, net GNDPWR
- added copper zone on F.Cu, net GNDPWR
Other:
- outline, holes or cut-outs redrawn
- board text added: "COM0"
- board text added: "COM1"
- board text added: "COM2"
- board text added: "COM3"
- board text added: "IN0+"
- board text added: "IN0-"
- board text added: "IN1+"
- board text added: "IN1-"
- board text added: "IN2+"
- board text added: "IN2-"
- board text added: "IN3+"
- board text added: "IN3-"
- board text added: "OA0"
- board text added: "OA1"
- board text added: "OA2"
- board text added: "OA3"
- board text added: "OB0"
- board text added: "OB1"
- board text added: "OB2"
- board text added: "OB3"
- board text added: "VDD0"
- board text added: "VDD1"
- board text added: "VDD2"
- board text added: "VDD3"
