File: Public/Module/ADS131M02/ADS131M02_KiCad/ADS131M02_KiCad.kicad_pcb (KiCad board)
At the start: 2 copper layers, 58.4 x 73.7 mm, 26 parts, among them J1 Power_Input, J2 Analog_Input, J3 Analog_Input, J4 Analog_Input, J5 Analog_Input, J6 Digital_IO, U1 ADS131M02_TSSOP20, U2 LP2985-3.3

Commit message: Update
Routing:
- net GNDREF: vias 1 -> 77
Changed lines of the file:
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@@
   (segment (start 120.3125 46.99) (end 115.365 46.99) (width 0.508) (layer "F.Cu") (net 2))
   (segment (start 127.635 46.99) (end 125.525 46.99) (width 0.508) (layer "F.Cu") (net 2))
+  (via (at 142.24 83.82) (size 0.8128) (drill 0.4064) (layers "F.Cu" "B.Cu") (free) (net 2))
+  (via (at 142.24 91.44) (size 0.8128) (drill 0.4064) (layers "F.Cu" "B.Cu") (free) (net 2))
+  (via (at 88.9 48.26) (size 0.8128) (drill 0.4064) (layers "F.Cu" "B.Cu") (free) (net 2))
+  (via (at 88.9 101.6) (size 0.8128) (drill 0.4064) (layers "F.Cu" "B.Cu") (free) (net 2))
+  (via (at 109.22 109.22) (size 0.8128) (drill 0.4064) (layers "F.Cu" "B.Cu") (free) (net 2))
+  (via (at 116.84 40.64) (size 0.8128) (drill 0.4064) (layers "F.Cu" "B.Cu") (free) (net 2))
+  (via (at 88.9 76.2) (size 0.8128) (drill 0.4064) (layers "F.Cu" "B.Cu") (free) (net 2))
+  (via (at 88.9 88.9) (size 0.8128) (drill 0.4064) (layers "F.Cu" "B.Cu") (free) (net 2))
+  (via (at 142.24 55.88) (size 0.8128) (drill 0.4064) (layers "F.Cu" "B.Cu") (free) (net 2))
+  (via (at 99.06 109.22) (size 0.8128) (drill 0.4064) (layers "F.Cu" "B.Cu") (free) (net 2))
+  (via (at 142.24 101.6) (size 0.8128) (drill 0.4064) (layers "F.Cu" "B.Cu") (free) (net 2))
+  (via (at 116.84 109.22) (size 0.8128) (drill 0.4064) (layers "F.Cu" "B.Cu") (free) (net 2))
+  (via (at 101.6 40.64) (size 0.8128) (drill 0.4064) (layers "F.Cu" "B.Cu") (free) (net 2))
+  (via (at 134.62 109.22) (size 0.8128) (drill 0.4064) (layers "F.Cu" "B.Cu") (free) (net 2))
+  (via (at 142.24 73.66) (size 0.8128) (drill 0.4064) (layers "F.Cu" "B.Cu") (free) (net 2))
+  (via (at 127 109.22) (size 0.8128) (drill 0.4064) (layers "F.Cu" "B.Cu") (free) (net 2))
+  (via (at 142.24 58.42) (size 0.8128) (drill 0.4064) (layers "F.Cu" "B.Cu") (free) (net 2))
+  (via (at 119.38 40.64) (size 0.8128) (drill 0.4064) (layers "F.Cu" "B.Cu") (free) (net 2))
+  (via (at 142.24 63.5) (size 0.8128) (drill 0.4064) (layers "F.Cu" "B.Cu") (free) (net 2))
+  (via (at 142.24 71.12) (size 0.8128) (drill 0.4064) (layers "F.Cu" "B.Cu") (free) (net 2))
+  (via (at 88.9 93.98) (size 0.8128) (drill 0.4064) (layers "F.Cu" "B.Cu") (free) (net 2))
+  (via (at 142.24 86.36) (size 0.8128) (drill 0.4064) (layers "F.Cu" "B.Cu") (free) (net 2))
+  (via (at 142.24 81.28) (size 0.8128) (drill 0.4064) (layers "F.Cu" "B.Cu") (free) (net 2))
+  (via (at 88.9 83.82) (size 0.8128) (drill 0.4064) (layers "F.Cu" "B.Cu") (free) (net 2))
+  (via (at 127 40.64) (size 0.8128) (drill 0.4064) (layers "F.Cu" "B.Cu") (free) (net 2))
+  (via (at 124.46 40.64) (size 0.8128) (drill 0.4064) (layers "F.Cu" "B.Cu") (free) (net 2))
+  (via (at 119.38 109.22) (size 0.8128) (drill 0.4064) (layers "F.Cu" "B.Cu") (free) (net 2))
+  (via (at 142.24 66.04) (size 0.8128) (drill 0.4064) (layers "F.Cu" "B.Cu") (free) (net 2))
+  (via (at 96.52 109.22) (size 0.8128) (drill 0.4064) (layers "F.Cu" "B.Cu") (free) (net 2))
+  (via (at 88.9 50.8) (size 0.8128) (drill 0.4064) (layers "F.Cu" "B.Cu") (free) (net 2))
+  (via (at 88.9 55.88) (size 0.8128) (drill 0.4064) (layers "F.Cu" "B.Cu") (free) (net 2))
+  (via (at 106.68 40.64) (size 0.8128) (drill 0.4064) (layers "F.Cu" "B.Cu") (free) (net 2))
+  (via (at 88.9 78.74) (size 0.8128) (drill 0.4064) (layers "F.Cu" "B.Cu") (free) (net 2))
+  (via (at 142.24 93.98) (size 0.8128) (drill 0.4064) (layers "F.Cu" "B.Cu") (free) (net 2))
+  (via (at 88.9 91.44) (size 0.8128) (drill 0.4064) (layers "F.Cu" "B.Cu") (free) (net 2))
+  (via (at 142.24 68.58) (size 0.8128) (drill 0.4064) (layers "F.Cu" "B.Cu") (free) (net 2))
+  (via (at 121.92 109.22) (size 0.8128) (drill 0.4064) (layers "F.Cu" "B.Cu") (free) (net 2))
+  (via (at 142.24 78.74) (size 0.8128) (drill 0.4064) (layers "F.Cu" "B.Cu") (free) (net 2))
+  (via (at 129.54 40.64) (size 0.8128) (drill 0.4064) (layers "F.Cu" "B.Cu") (free) (net 2))
+  (via (at 111.76 40.64) (size 0.8128) (drill 0.4064) (layers "F.Cu" "B.Cu") (free) (net 2))
+  (via (at 88.9 71.12) (size 0.8128) (drill 0.4064) (layers "F.Cu" "B.Cu") (free) (net 2))
+  (via (at 132.08 109.22) (size 0.8128) (drill 0.4064) (layers "F.Cu" "B.Cu") (free) (net 2))
+  (via (at 142.24 50.8) (size 0.8128) (drill 0.4064) (layers "F.Cu" "B.Cu") (free) (net 2))
+  (via (at 114.3 40.64) (size 0.8128) (drill 0.4064) (layers "F.Cu" "B.Cu") (free) (net 2))
+  (via (at 88.9 58.42) (size 0.8128) (drill 0.4064) (layers "F.Cu" "B.Cu") (free) (net 2))
+  (via (at 111.76 109.22) (size 0.8128) (drill 0.4064) (layers "F.Cu" "B.Cu") (free) (net 2))
+  (via (at 88.9 96.52) (size 0.8128) (drill 0.4064) (layers "F.Cu" "B.Cu") (free) (net 2))
+  (via (at 109.22 40.64) (size 0.8128) (drill 0.4064) (layers "F.Cu" "B.Cu") (free) (net 2))
+  (via (at 106.68 109.22) (size 0.8128) (drill 0.4064) (layers "F.Cu" "B.Cu") (free) (net 2))
+  (via (at 88.9 60.96) (size 0.8128) (drill 0.4064) (layers "F.Cu" "B.Cu") (free) (net 2))
+  (via (at 104.14 109.22) (size 0.8128) (drill 0.4064) (layers "F.Cu" "B.Cu") (free) (net 2))
+  (via (at 88.9 53.34) (size 0.8128) (drill 0.4064) (layers "F.Cu" "B.Cu") (free) (net 2))
+  (via (at 142.24 88.9) (size 0.8128) (drill 0.4064) (layers "F.Cu" "B.Cu") (free) (net 2))
+  (via (at 99.06 40.64) (size 0.8128) (drill 0.4064) (layers "F.Cu" "B.Cu") (free) (net 2))
+  (via (at 96.52 40.64) (size 0.8128) (drill 0.4064) (layers "F.Cu" "B.Cu") (free) (net 2))
+  (via (at 88.9 68.58) (size 0.8128) (drill 0.4064) (layers "F.Cu" "B.Cu") (free) (net 2))
+  (via (at 88.9 86.36) (size 0.8128) (drill 0.4064) (layers "F.Cu" "B.Cu") (free) (net 2))
+  (via (at 101.6 109.22) (size 0.8128) (drill 0.4064) (layers "F.Cu" "B.Cu") (free) (net 2))
   (via (at 127.635 46.99) (size 1.2192) (drill 0.6096) (layers "F.Cu" "B.Cu") (free) (net 2))
+  (via (at 142.24 96.52) (size 0.8128) (drill 0.4064) (layers "F.Cu" "B.Cu") (free) (net 2))
+  (via (at 134.62 40.64) (size 0.8128) (drill 0.4064) (layers "F.Cu" "B.Cu") (free) (net 2))
+  (via (at 121.92 40.64) (size 0.8128) (drill 0.4064) (layers "F.Cu" "B.Cu") (free) (net 2))
+  (via (at 142.24 53.34) (size 0.8128) (drill 0.4064) (layers "F.Cu" "B.Cu") (free) (net 2))
+  (via (at 114.3 109.22) (size 0.8128) (drill 0.4064) (layers "F.Cu" "B.Cu") (free) (net 2))
+  (via (at 124.46 109.22) (size 0.8128) (drill 0.4064) (layers "F.Cu" "B.Cu") (free) (net 2))
+  (via (at 142.24 60.96) (size 0.8128) (drill 0.4064) (layers "F.Cu" "B.Cu") (free) (net 2))
+  (via (at 142.24 99.06) (size 0.8128) (drill 0.4064) (layers "F.Cu" "B.Cu") (free) (net 2))
+  (via (at 88.9 99.06) (size 0.8128) (drill 0.4064) (layers "F.Cu" "B.Cu") (free) (net 2))
+  (via (at 88.9 81.28) (size 0.8128) (drill 0.4064) (layers "F.Cu" "B.Cu") (free) (net 2))
+  (via (at 142.24 76.2) (size 0.8128) (drill 0.4064) (layers "F.Cu" "B.Cu") (free) (net 2))
+  (via (at 88.9 66.04) (size 0.8128) (drill 0.4064) (layers "F.Cu" "B.Cu") (free) (net 2))
+  (via (at 132.08 40.64) (size 0.8128) (drill 0.4064) (layers "F.Cu" "B.Cu") (free) (net 2))
+  (via (at 88.9 63.5) (size 0.8128) (drill 0.4064) (layers "F.Cu" "B.Cu") (free) (net 2))
+  (via (at 129.54 109.22) (size 0.8128) (drill 0.4064) (layers "F.Cu" "B.Cu") (free) (net 2))
+  (via (at 142.24 48.26) (size 0.8128) (drill 0.4064) (layers "F.Cu" "B.Cu") (free) (net 2))
+  (via (at 104.14 40.64) (size 0.8128) (drill 0.4064) (layers "F.Cu" "B.Cu") (free) (net 2))
+  (via (at 88.9 73.66) (size 0.8128) (drill 0.4064) (layers "F.Cu" "B.Cu") (free) (net 2))
   (segment (start 118.0375 46.04) (end 118.0375 45.0125) (width 0.254) (layer "F.Cu") (net 3))
   (segment (start 117.065 44.04) (end 115.365 44.04) (width 0.254) (layer "F.Cu") (net 3))
